File: pcb/dd2702h-interface.kicad_pcb (KiCad board)
At the start: 2 copper layers, 33 x 33 mm, 13 parts, among them J1 Conn_01x11_Pin, Q1 2N3904, Q2 2N3904, Q3 2N3904, Q4 2N3904, Q5 2N3904, U1 WeMos_D1_mini

Commit message: Mounting holes; autorouted
Parts:
- added REF**: MountingHole_2mm, MountingHole:MountingHole_2mm, F.Cu at (116.8, 71.1)
- added REF**: MountingHole_2mm, MountingHole:MountingHole_2mm, F.Cu at (88.9, 71.1)
- added REF**: MountingHole_2mm, MountingHole:MountingHole_2mm, F.Cu at (116.8, 99.1)
Routing:
- net Net-(Q4-B): track 20.1 -> 10.6 mm
- net DOWN_E: track 26.0 -> 22.5 mm
- net CH_UP_E: track 25.3 -> 23.1 mm
- net GPIO13: track 10.4 -> 11.9 mm
- net GPIO12: track 10.1 -> 11.6 mm
- net GPIO14: track 9.86 -> 11.4 mm
- net CH_DOWN_E: track 24.5 -> 23.2 mm
- net DOWN_C: track 20.8 -> 19.5 mm
- net STOP_E: track 24.7 -> 23.5 mm
- net Net-(Q2-B): track 10.3 -> 11.5 mm
- net CH_DOWN_C: track 20.6 -> 19.8 mm
- net GPIO15: track 10.7 -> 11.3 mm
- net GPIO2: track 16.4 -> 17.1 mm
- net Net-(Q5-B): track 12.3 -> 11.7 mm
- net Net-(Q3-B): track 11.0 -> 10.4 mm
Other:
- board text added: "HA DD2702H v0.2"
- board text removed: "HA DD2702H v0.1"
